File: 16_led_array.kicad_pcb (KiCad board)
At the start: 2 copper layers, 61.6 x 47 mm, 36 parts, among them J1 Conn_01x05, U1 74HC595, U2 74HC595

Commit message: Final layout
Signed-off-by: Richard Memory <richardfmemory@gmail.com>
Parts:
- added G***: LOGO, graphics:logo, F.Cu at (142.2, 57.1)
- added G***: LOGO, graphics:logo, F.Cu at (141.6, 54.0)
- added G***: LOGO, graphics:logo, F.Cu at (142.2, 53.3)
- added G***: LOGO, graphics:logo, F.Cu at (144.1, 54.0)
- added G***: LOGO, graphics:logo, F.Cu at (140.3, 54.6)
- added G***: LOGO, graphics:logo, F.Cu at (201.9, 47.6)
- added G***: LOGO, graphics:logo, F.Cu at (200.0, 52.7)
Routing:
- net VCC: track 0.00 -> 164.5 mm
- net GND: track 0.00 -> 53.4 mm, vias 0 -> 1
- net /led_2_8: track 0.00 -> 35.5 mm, vias 0 -> 2
- net /led_1_8: track 0.00 -> 34.5 mm, vias 0 -> 2
- net /led_2_7: track 0.00 -> 33.9 mm, vias 0 -> 2
- net /led_1_1: track 0.00 -> 33.1 mm, vias 0 -> 4
- net /led_2_6: track 0.00 -> 33.1 mm, vias 0 -> 2
- net /CLOCK: track 0.00 -> 31.8 mm, vias 0 -> 2
- net /led_1_7: track 0.00 -> 30.7 mm, vias 0 -> 2
- net /led_2_5: track 0.00 -> 30.4 mm, vias 0 -> 2
- net /LATCH: track 0.00 -> 27.5 mm, vias 0 -> 2
- net /led_2_3: track 0.00 -> 26.6 mm, vias 0 -> 2
- net /led_1_6: track 0.00 -> 26.3 mm, vias 0 -> 2
- net /led_2_4: track 0.00 -> 26.2 mm, vias 0 -> 2
- net /led_2_2: track 0.00 -> 26.2 mm, vias 0 -> 2
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- added copper zone on B.Cu, net GND
- added copper zone on F.Cu, net VCC
Other:
- board text added: "16-LED board with shift registers"
- board text added: "V1.0"
